Commit message: Added some indicators on wheels to view rotation

File: src/atom/urdf/atom.xacro (robot description, xacro)
@@ -61,4 +61,25 @@
 		</collision>
 	</link>
+	<!-- Cube -->
+	<!-- <link name="cube_link">
+		<inertial>
+			<mass value="0.0"/>
+			<origin xyz="0 ${robot_wheel_radius} 0"/>
+			<inertia
+				ixx="0.0" ixy="0.0" ixz="0.0"
+				iyy="0.0" iyz="0.0"
+				izz="0.0"
+			/>
+		</inertial>
+		<visual>
+			<origin xyz="0 0 0"/>
+			<geometry>
+				<box size="${robot_wheel_radius} 20 5"/>
+			</geometry>
+		</visual>
+		<collision>
+			<origin xyz="0 0 0"/>
+		</collision>
+	</link> -->
 	<!-- Right Wheel Front-->
 	<link name="right_wheel_front">
@@ -154,4 +175,100 @@
 			<geometry>
 				<box size="0.05 0.05 0.05"/>
+			</geometry>
+		</collision>
+	</link>
+    <!-- Front Left Indicator -->
+	<link name="front_left_indicator">
+		<inertial>
+			<mass value="0"/>
+			<origin xyz="0 0 0" rpy="0 0 0"/>
+			<inertia
+		        ixx="1e-6" ixy="0.0" ixz="0.0"
+		        iyy="1e-6" iyz="0.0"
+		        izz="1e-6"
+		      />
+		</inertial>
+		<visual>
+			<origin xyz="0 0 0" rpy="0 0 0"/>
+			<geometry>
+				<box size="${robot_wheel_radius} 0.05 0.05"/>
+			</geometry>
+		</visual>
+		<collision>
+			<origin xyz="0 0 0" rpy="0 0 0"/>
+			<geometry>
+				<box size="0.0 0.0 0.0"/>
+			</geometry>
+		</collision>
+	</link>
+    <!-- Front Right Indicator -->
+	<link name="front_right_indicator">
+		<inertial>
+			<mass value="0"/>
+			<origin xyz="0 0 0" rpy="0 0 0"/>
+			<inertia
+		        ixx="1e-6" ixy="0.0" ixz="0.0"
+		        iyy="1e-6" iyz="0.0"
+		        izz="1e-6"
+		      />
+		</inertial>
+		<visual>
+			<origin xyz="0 0 0" rpy="0 0 0"/>
+			<geometry>
+				<box size="${robot_wheel_radius} 0.05 0.05"/>
+			</geometry>
+		</visual>
+		<collision>
+			<origin xyz="0 0 0" rpy="0 0 0"/>
+			<geometry>
+				<box size="0.0 0.0 0.0"/>
+			</geometry>
+		</collision>
+	</link>
+	<!-- Back Left Indicator -->
+	<link name="back_left_indicator">
+		<inertial>
+			<mass value="0"/>
+			<origin xyz="0 0 0" rpy="0 0 0"/>
+			<inertia
+		        ixx="1e-6" ixy="0.0" ixz="0.0"
+		        iyy="1e-6" iyz="0.0"
+		        izz="1e-6"
+		      />
+		</inertial>
+		<visual>
+			<origin xyz="0 0 0" rpy="0 0 0"/>
+			<geometry>
+				<box size="${robot_wheel_radius} 0.05 0.05"/>
+			</geometry>
+		</visual>
+		<collision>
+			<origin xyz="0 0 0" rpy="0 0 0"/>
+			<geometry>
+				<box size="0.0 0.0 0.0"/>
+			</geometry>
+		</collision>
+	</link>
+	<!-- Back Right Indicator -->
+	<link name="back_right_indicator">
+		<inertial>
+			<mass value="0"/>
+			<origin xyz="0 0 0" rpy="0 0 0"/>
+			<inertia
+		        ixx="1e-6" ixy="0.0" ixz="0.0"
+		        iyy="1e-6" iyz="0.0"
+		        izz="1e-6"
+		      />
+		</inertial>
+		<visual>
+			<origin xyz="0 0 0" rpy="0 0 0"/>
+			<geometry>
+				<box size="${robot_wheel_radius} 0.05 0.05"/>
+			</geometry>
+		</visual>
+		<collision>
+			<origin xyz="0 0 0" rpy="0 0 0"/>
+			<geometry>
+				<box size="0.0 0.0 0.0"/>
 			</geometry>
 		</collision>
@@ -239,4 +356,28 @@
 		<child link="chassis" />
 	</joint>
+    <joint name="front_left_indicator_joint" type="fixed">
+	    <origin xyz="0 0.02 0" rpy="0 0 0" />
+	    <parent link="left_wheel_front"/>
+	    <child link="front_left_indicator" />
+	    <axis xyz="0 0 0"/>
+	</joint>
+ 	<joint name="front_right_indicator_joint" type="fixed">
+	    <origin xyz="0 -0.02 0" rpy="0 0 0" />
+	    <parent link="right_wheel_front"/>
+	    <child link="front_right_indicator" />
+	    <axis xyz="0 0 0"/>
+	</joint>
+	<joint name="back_left_indicator_joint" type="fixed">
+	    <origin xyz="0 0.02 0" rpy="0 0 0" />
+	    <parent link="left_wheel_back"/>
+	    <child link="back_left_indicator" />
+	    <axis xyz="0 0 0"/>
+	</joint>
+ 	<joint name="back_right_indicator_joint" type="fixed">
+	    <origin xyz="0 -0.02 0" rpy="0 0 0" />
+	    <parent link="right_wheel_back"/>
+	    <child link="back_right_indicator" />
+	    <axis xyz="0 0 0"/>
+	</joint>
 	<!-- Color of bot -->
 	<gazebo reference="left_wheel_front">
@@ -285,4 +426,16 @@
 		<material>Gazebo/Blue</material>
 	</gazebo>
+	<gazebo reference="front_left_indicator">
+		<material>Gazebo/Yellow</material>
+	</gazebo>
+	<gazebo reference="front_right_indicator">
+		<material>Gazebo/Yellow</material>
+	</gazebo>
+	<gazebo reference="back_left_indicator">
+		<material>Gazebo/Yellow</material>
+	</gazebo>
+	<gazebo reference="back_right_indicator">
+		<material>Gazebo/Yellow</material>
+	</gazebo>
 	<gazebo>
 		<plugin name="control_plugin" filename="libcontrol_plugin.so"/>

Commit message: Cleanup & comments

File: src/atom/urdf/atom.xacro (robot description, xacro)
@@ -417,7 +417,4 @@
 		<minDepth>0.00</minDepth>
 	</gazebo>
-	<!--<gazebo reference="right_wheel">
-		<material>Gazebo/Green</material>
-	</gazebo>-->
 	<gazebo reference="camera">
 		<material>Gazebo/Red</material>
@@ -438,7 +435,4 @@
 		<material>Gazebo/Yellow</material>
 	</gazebo>
-	<!-- <gazebo>
-		<plugin name="control_plugin" filename="libcontrol_plugin.so"/>
-	</gazebo> -->
 	<!-- Motor, Camera and Lidar Simulation -->
 	<xacro:include filename="$(find atom)/urdf/atom.gazebo" />
